File: controller_board/controller_board.kicad_pcb (KiCad board)
At the start: 2 copper layers, 0 parts

Commit message: PCB-now
Parts:
- added C1: 1u, Capacitor_THT:C_Disc_D5.0mm_W2.5mm_P5.00mm, F.Cu at (30.4, 17.6)
- added C2: 1u, Capacitor_THT:C_Disc_D5.0mm_W2.5mm_P5.00mm, F.Cu at (21.2, 24.9)
- added D1: LED, LED_THT:LED_D3.0mm, F.Cu at (16.3, 29.1)
- added D2: LED, LED_THT:LED_D3.0mm, F.Cu at (38.4, 91.9)
- added D3: LED, LED_THT:LED_D3.0mm, F.Cu at (43.6, 91.9)
- added J1: Jack-DC, MyLib:DCJack2.1, F.Cu at (38.8, 26.1)
- added R1: 20k, Resistor_THT:R_Axial_DIN0204_L3.6mm_D1.6mm_P7.62mm_Horizontal, F.Cu at (30.1, 83.6)
- added R2: 20k, Resistor_THT:R_Axial_DIN0204_L3.6mm_D1.6mm_P7.62mm_Horizontal, F.Cu at (33.2, 83.6)
- added R3: 4.7K, Resistor_THT:R_Axial_DIN0204_L3.6mm_D1.6mm_P7.62mm_Horizontal, F.Cu at (29.3, 29.1)
- added R4: 4.7K, Resistor_THT:R_Axial_DIN0204_L3.6mm_D1.6mm_P7.62mm_Horizontal, F.Cu at (36.2, 76.0)
- added R5: 4.7K, Resistor_THT:R_Axial_DIN0204_L3.6mm_D1.6mm_P7.62mm_Horizontal, F.Cu at (39.4, 76.0)
- added R6: 1k, Resistor_THT:R_Axial_DIN0204_L3.6mm_D1.6mm_P7.62mm_Horizontal, F.Cu at (42.5, 76.0)
- added REF**: MountingHole_3.2mm_M3, MountingHole:MountingHole_3.2mm_M3, F.Cu at (19.0, 91.0)
- added REF**: MountingHole_3.2mm_M3, MountingHole:MountingHole_3.2mm_M3, F.Cu at (19.0, 19.0)
- added REF**: MountingHole_3.2mm_M3, MountingHole:MountingHole_3.2mm_M3, F.Cu at (61.0, 19.0)
- added REF**: MountingHole_3.2mm_M3, MountingHole:MountingHole_3.2mm_M3, F.Cu at (61.0, 91.0)
- added RV1: ~, MyLib:VR-sliderV2, F.Cu at (51.0, 55.0)
- added SW1: SW_Push, Connector_PinHeader_2.54mm:PinHeader_1x02_P2.54mm_Vertical, F.Cu at (28.8, 90.3)
- added SW2: SW_Push, Connector_PinHeader_2.54mm:PinHeader_1x02_P2.54mm_Vertical, F.Cu at (32.6, 90.3)
- added U1: XIAO_ESP32C3, MyLib:XIAO_ESP32C3, F.Cu at (25.9, 44.9)
- added U2: LM1117GS-3.3, Package_TO_SOT_SMD:SOT-223-3_TabPin2, F.Cu at (27.2, 23.9)
- added U3: OSL10564, MyLib:OSL10564-MODULE, F.Cu at (21.6, 73.1)
Routing:
- net +3.3V: track 0.00 -> 148.9 mm, vias 0 -> 1
- net LATCH: track 0.00 -> 57.3 mm
- net Volume: track 0.00 -> 55.1 mm
- net DirectionSW: track 0.00 -> 40.1 mm
- net LEDSW: track 0.00 -> 40.0 mm
- net SCK: track 0.00 -> 31.0 mm, vias 0 -> 1
- net +BATT: track 0.00 -> 26.4 mm
- net MOSI: track 0.00 -> 26.3 mm
- net LED: track 0.00 -> 25.8 mm
- net Net-(D3-A): track 0.00 -> 9.01 mm
- net Net-(D2-A): track 0.00 -> 8.44 mm
- net Net-(R6-Pad2): track 0.00 -> 8.36 mm
- net Net-(D1-A): track 0.00 -> 2.82 mm
- net GND: vias 0 -> 76
- added copper zone on B.Cu, net GND
- added copper zone on F.Cu, net GND
Other:
- board outline added: 50 x 80 mm
- board text added: "3.3V"
- board text added: "LED"
- board text added: "VCC"
